Commit message: Fix positio origin

File: urdf/carver.urdf (robot description, URDF)
Before this commit: robot carver_description, 14 links, 13 joints
Joints:
- joint world_base_joint: origin xyz=0 0 0 rpy=0 0 0 -> xyz=0 0 0.345 rpy=0 0 0

Commit message: edit urdf

File: urdf/carver.urdf (robot description, URDF)
Before this commit: robot carver_description, 14 links, 13 joints
Links:
- removed link RPLIDAR_B_Link
- removed link RPLIDAR_F_Link
- added link IMU_L_Link, mass 0.000983130183652038; collision mesh filename=package://carver_description/meshes/IMU_L_Link.STL; visual mesh filename=package://carver_description/meshes/IMU_L_Link.STL
- added link IMU_R_Link, mass 0.000983130183652042; collision mesh filename=package://carver_description/meshes/IMU_R_Link.STL; visual mesh filename=package://carver_description/meshes/IMU_R_Link.STL
- added link RPLIDAR_LB_Link, mass 0.0327576849816352; collision mesh filename=package://carver_description/meshes/RPLIDAR_LB_Link.STL; visual mesh filename=package://carver_description/meshes/RPLIDAR_LB_Link.STL
- added link RPLIDAR_LF_Link, mass 0.0327576849285788; collision mesh filename=package://carver_description/meshes/RPLIDAR_LF_Link.STL; visual mesh filename=package://carver_description/meshes/RPLIDAR_LF_Link.STL
- added link RPLIDAR_RB_Link, mass 0.0327576843712563; collision mesh filename=package://carver_description/meshes/RPLIDAR_RB_Link.STL; visual mesh filename=package://carver_description/meshes/RPLIDAR_RB_Link.STL
- link L515_Link: mass 0.0519003008836609 -> 0.0519003008833496
- link LD_SICK_Link: mass 0.911976961838327 -> 0.911976961838331
- link T265_Link: mass 0.0153522629827051 -> 0.0153522629829022
- link base_link: mass 363.855564635503 -> 223.870769479693
Joints:
- removed joint base_RPLIDAR_F_joint
- removed joint base_RPLIDAR_joint
- added joint base_IMU_L_joint: type fixed, parent base_link, child IMU_L_Link, origin xyz=0.029419441223861 0.0191387564081886 0.383 rpy=0 0 0, axis 0 0 0
- added joint base_IMU_R_joint: type fixed, parent base_link, child IMU_R_Link, origin xyz=0.0271694412238607 -0.0191012435918216 0.383 rpy=0 0 0, axis 0 0 0
- added joint base_RPLIDAR_LB_joint: type fixed, parent base_link, child RPLIDAR_LB_Link, origin xyz=-0.894118330232296 0.316260936090295 0.0854783318747023 rpy=0 0 0, axis 0 0 0
- added joint base_RPLIDAR_LF_joint: type fixed, parent base_link, child RPLIDAR_LF_Link, origin xyz=0.912928672596467 0.374905020086834 0.0854783318747023 rpy=0 0 0, axis 0 0 0
- added joint base_RPLIDAR_RB_joint: type fixed, parent base_link, child RPLIDAR_RB_Link, origin xyz=-0.866459374365379 -0.3462959068844 0.0854783318747023 rpy=0 0 0, axis 0 0 0
- joint base_C16_joint: origin xyz=0.237767026438175 0 1.56788196587258 rpy=0 0 0 -> xyz=0.237767026438191 0 1.56788196587259 rpy=0 0 0
- joint base_L515_joint: origin xyz=0.926668924633506 -1.17161568835617E-05 0.153229231648557 rpy=0 0 0 -> xyz=0.929717002207267 -1.17161560733146E-05 -0.0149951470092575 rpy=0 0 0
- joint base_LD_SICK_joint: origin xyz=1.04931892463351 0 -0.0799999999999999 rpy=0 0 0 -> xyz=0.942318924633513 0 0.215 rpy=0 0 0

Commit message: add_RF_lidar

File: urdf/carver.urdf (robot description, URDF)
Before this commit: robot carver_description, 17 links, 16 joints
Links:
- added link RPLIDAR_RF_Link, mass 0.0327576849297121; collision mesh filename=package://carver_description/meshes/RPLIDAR_RF_Link.STL; visual mesh filename=package://carver_description/meshes/RPLIDAR_RF_Link.STL
- link RPLIDAR_LB_Link: mass 0.0327576849816352 -> 0.0327576849816269
- link RPLIDAR_LF_Link: mass 0.0327576849285788 -> 0.0327576849285776
- link RPLIDAR_RB_Link: mass 0.0327576843712563 -> 0.0327576843712578
- link base_link: mass 223.870769479693 -> 223.948097033883
Joints:
- added joint base_RPLIDAR_RF_joint: type fixed, parent base_link, child RPLIDAR_RF_Link, origin xyz=0.912928672596467 -0.374905020086827 0.0854783318747024 rpy=0 0 0, axis 0 0 0

Commit message: fix lidar

File: urdf/carver.urdf (robot description, URDF)
Before this commit: robot carver_description, 18 links, 17 joints
Links:
- removed link RPLIDAR_LF_Link
- removed link RPLIDAR_RB_Link
- link IMU_R_Link: mass 0.000983130183652042 -> 0.000983130183652043
- link LD_SICK_Link: mass 0.911976961838331 -> 0.911976961838319
- link RPLIDAR_LB_Link: mass 0.0327576849816269 -> 0.0328083847884949
- link RPLIDAR_RF_Link: mass 0.0327576849297121 -> 0
- link T265_Link: mass 0.0153522629829022 -> 0.015352262982903
- link base_link: mass 223.948097033883 -> 224.416537318038
- link front_right_wheel_Link: mass 5.024500013847 -> 5.0245
Joints:
- removed joint base_RPLIDAR_LF_joint
- removed joint base_RPLIDAR_RB_joint
- joint base_C16_joint: origin xyz=0.237767026438191 0 1.56788196587259 rpy=0 0 0 -> xyz=0.23777 0 1.5679 rpy=0 0 0
- joint base_IMU_L_joint: origin xyz=0.029419441223861 0.0191387564081886 0.383 rpy=0 0 0 -> xyz=0.029419 0.019139 0.383 rpy=0 0 0
- joint base_IMU_R_joint: origin xyz=0.0271694412238607 -0.0191012435918216 0.383 rpy=0 0 0 -> xyz=0.027169 -0.019101 0.383 rpy=0 0 0
- joint base_L515_joint: origin xyz=0.929717002207267 -1.17161560733146E-05 -0.0149951470092575 rpy=0 0 0 -> xyz=0.92972 -1.1716E-05 -0.014995 rpy=0 0 0
- joint base_LD_SICK_joint: origin xyz=0.942318924633513 0 0.215 rpy=0 0 0 -> xyz=0.94232 0 0.215 rpy=0 0 0
- joint base_RPLIDAR_LB_joint: origin xyz=-0.894118330232296 0.316260936090295 0.0854783318747023 rpy=0 0 0 -> xyz=-0.85116 0.34072 0.085015 rpy=0 0 3.1412
- joint base_RPLIDAR_RF_joint: origin xyz=0.912928672596467 -0.374905020086827 0.0854783318747024 rpy=0 0 0 -> xyz=0.91252 -0.38133 0.15392 rpy=0 0 0
- joint base_T265_joint: origin xyz=0.914568924633506 0.000699999999822833 0.423999999999455 rpy=0 0 0 -> xyz=0.91457 0.0007 0.424 rpy=0 0 0
- joint base_rear_left_wheel_joint: origin xyz=-0.636881075366491 0.3955 -0.17 rpy=-1.5707963267949 0 0 -> xyz=-0.63688 0.3955 -0.17 rpy=-1.5708 0 0
- joint base_rear_right_wheel_joint: origin xyz=-0.636881075366491 -0.3955 -0.17 rpy=-1.5707963267949 0 0 -> xyz=-0.63688 -0.3955 -0.17 rpy=-1.5708 0 0
- joint front_left_steering_front_left_wheel_joint: axis 0.036417508182449 0 -0.999336662540598 -> 0.036418 0 -0.99934; origin xyz=-0.00404234340824972 0.110926369542007 -0.0112500000000002 rpy=-1.5707963267949 0 0 -> xyz=-0.0040423 0.11093 -0.01125 rpy=-1.5708 0 0

Commit message: add base under back lidar

File: urdf/carver.urdf (robot description, URDF)
Before this commit: robot carver_description, 16 links, 15 joints
Links:
- link IMU_R_Link: mass 0.000983130183652043 -> 0.000983130183652042
- link LD_SICK_Link: mass 0.911976961838319 -> 0.911976961838322
- link RPLIDAR_LB_Link: mass 0.0328083847884949 -> 0.0328083847884842
- link RPLIDAR_RF_Link: mass 0 -> 0.0328083843446528
- link base_link: mass 224.416537318038 -> 224.620223914356
- link front_right_wheel_Link: mass 5.0245 -> 5.024500013847
Joints:
- joint base_C16_joint: origin xyz=0.23777 0 1.5679 rpy=0 0 0 -> xyz=0.237767026438191 0 1.56788196587259 rpy=0 0 0
- joint base_IMU_L_joint: origin xyz=0.029419 0.019139 0.383 rpy=0 0 0 -> xyz=0.029419441223861 0.0191387564081886 0.383 rpy=0 0 0
- joint base_IMU_R_joint: origin xyz=0.027169 -0.019101 0.383 rpy=0 0 0 -> xyz=0.0271694412238607 -0.0191012435918216 0.383 rpy=0 0 0
- joint base_L515_joint: origin xyz=0.92972 -1.1716E-05 -0.014995 rpy=0 0 0 -> xyz=0.929717002207267 -1.17161560733146E-05 -0.0149951470092575 rpy=0 0 0
- joint base_LD_SICK_joint: origin xyz=0.94232 0 0.215 rpy=0 0 0 -> xyz=0.942318924633513 0 0.215 rpy=0 0 0
- joint base_RPLIDAR_LB_joint: origin xyz=-0.85116 0.34072 0.085015 rpy=0 0 3.1412 -> xyz=-0.851155901465486 0.34071809177296 0.154015 rpy=0 0 3.14124991984497
- joint base_RPLIDAR_RF_joint: origin xyz=0.91252 -0.38133 0.15392 rpy=0 0 0 -> xyz=0.912523944720348 -0.381327891424126 0.153915 rpy=0 0 0
- joint base_T265_joint: origin xyz=0.91457 0.0007 0.424 rpy=0 0 0 -> xyz=0.914568924633506 0.000699999999822833 0.423999999999455 rpy=0 0 0
- joint base_rear_left_wheel_joint: origin xyz=-0.63688 0.3955 -0.17 rpy=-1.5708 0 0 -> xyz=-0.636881075366491 0.3955 -0.17 rpy=-1.5707963267949 0 0
- joint base_rear_right_wheel_joint: origin xyz=-0.63688 -0.3955 -0.17 rpy=-1.5708 0 0 -> xyz=-0.636881075366491 -0.3955 -0.17 rpy=-1.5707963267949 0 0
- joint front_left_steering_front_left_wheel_joint: axis 0.036418 0 -0.99934 -> 0.036417508182449 0 -0.999336662540598; origin xyz=-0.0040423 0.11093 -0.01125 rpy=-1.5708 0 0 -> xyz=-0.00404234340824972 0.110926369542007 -0.0112500000000002 rpy=-1.5707963267949 0 0

Commit message: add laser frame

File: urdf/carver.urdf (robot description, URDF)
Before this commit: robot carver_description, 16 links, 15 joints
Links:
- added link laser
Joints:
- removed joint base_RPLIDAR_LB_joint
- removed joint base_RPLIDAR_RF_joint
- added joint base_laser_joint: type fixed, parent base_link, child laser, origin xyz=0 0 0.154015 rpy=0 0 0
- added joint laser_RPLIDAR_LB_joint: type fixed, parent laser, child RPLIDAR_LB_Link, origin xyz=-0.851155901465486 0.34071809177296 0 rpy=0 0 3.14124991984497, axis 0 0 0
- added joint laser_RPLIDAR_RF_joint: type fixed, parent laser, child RPLIDAR_RF_Link, origin xyz=0.912523944720348 -0.381327891424126 0 rpy=0 0 0, axis 0 0 0

Commit message: Update carver.urdf

File: urdf/carver.urdf (robot description, URDF)
Before this commit: robot carver_description, 17 links, 16 joints
Links:
- removed link world
- added link base_footprint
Joints:
- joint world_base_joint: parent world -> base_footprint

Commit message: add gps link

File: urdf/carver.urdf (robot description, URDF)
Before this commit: robot carver_description, 17 links, 16 joints
Links:
- added link GPS_Link, mass 0.157649586184773; collision mesh filename=package://carver_description/meshes/GPS_Link.STL; visual mesh filename=package://carver_description/meshes/GPS_Link.STL
Joints:
- added joint base_GPS_joint: type fixed, parent base_link, child GPS_Link, origin xyz=0.23423178728353 0.373617987041938 1.499 rpy=0 0 0, axis 0 0 0
